File: Eagle/Power Supply Rev G.brd (EAGLE design)
At the start: 35 x 35 mm, 19 parts, among them J1 694106301002, J2 61300211121, J4 61300211121, J5 61300211121, U1 LM317

Commit message: changes to BOM for manufacturing
Parts:
- C1: value 100n -> 220n
Other:
- board text added: "Q-PCB-001 – Power Supply"
- board text removed: "Q-PCB-001 – 9V Battery"
Changed lines of the file:
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@@
 </layers>
 <board>
-<fusionsync huburn="a.YnVzaW5lc3M6cXVhbnR1bWh0aQ" projecturn="a.YnVzaW5lc3M6cXVhbnR1bWh0aSMyMDIwMDUxOTI5OTUwMjAwMQ" f3durn="urn:adsk.wipprod:dm.lineage:nuA8EwR3Q5KwxrhtXih1oQ" pcbguid="" lastpulledtime="" lastsyncedchangeguid="" latestrevisionid="3d818803-2117-49f3-8dad-6dd10c85da2e" lastsyncedrevisionid="3d818803-2117-49f3-8dad-6dd10c85da2e" lastboardhashguid="9cec1567-dc3f-ee4f-49be-c045e1c95a98" lastpushedtime="2020-08-01T22:58:15Z" linktopcb3d="true"/>
+<fusionsync huburn="a.YnVzaW5lc3M6cXVhbnR1bWh0aQ" projecturn="a.YnVzaW5lc3M6cXVhbnR1bWh0aSMyMDIwMDUxOTI5OTUwMjAwMQ" f3durn="urn:adsk.wipprod:dm.lineage:nuA8EwR3Q5KwxrhtXih1oQ" pcbguid="" lastpulledtime="" lastsyncedchangeguid="" latestrevisionid="3d818803-2117-49f3-8dad-6dd10c85da2e" lastsyncedrevisionid="3d818803-2117-49f3-8dad-6dd10c85da2e" lastboardhashguid="9cec1567-dc3f-ee4f-49be-c045e1c95a98" lastpushedtime="2020-08-01T22:58:15Z" linktopcb3d="false"/>
 <plain>
 <wire x1="0" y1="1" x2="0" y2="34" width="0.1524" layer="20"/>
 <text x="28.56" y="9.06" size="1.27" layer="26" ratio="10" rot="MR0">Rev G</text>
 <text x="28.56" y="11" size="1.27" layer="26" ratio="10" rot="MR0">TL</text>
-<text x="28.56" y="12.936" size="1.27" layer="26" ratio="10" rot="MR180" align="top-right">Q-PCB-001 – 9V Battery</text>
+<text x="29.36" y="12.836" size="1.27" layer="26" ratio="10" rot="MR180" align="top-right">Q-PCB-001 – Power Supply</text>
 <text x="22.6" y="3.2" size="1.27" layer="25" ratio="10">GND</text>
 <text x="30.3" y="8.8" size="1.27" layer="25" ratio="10">GND</text>
@@
 <attribute name="VALUE" x="11.333" y="6.833" size="1.27" layer="27" ratio="10" rot="R270"/>
 </element>
-<element name="C1" library="Quantum Projects" library_urn="urn:adsk.eagle:library:19630877" package="E2-4" package3d_urn="urn:adsk.eagle:package:21734552/2" value="100n" x="21" y="9.5" smashed="yes" rot="R270">
+<element name="C1" library="Quantum Projects" library_urn="urn:adsk.eagle:library:19630877" package="E2-4" package3d_urn="urn:adsk.eagle:package:21734552/2" value="220n" x="21" y="9.5" smashed="yes" rot="R270">
 <attribute name="NAME" x="24.4" y="10" size="1.27" layer="25" ratio="10" align="center"/>
 <attribute name="VALUE" x="18.46" y="6.833" size="1.27" layer="27" ratio="10" rot="R270"/>
